File: SWD_Debug.kicad_sch (KiCad schematic)
At the start: 1 part, among them J2 TC2030

Commit message: Push current KiCad workspace changes
Connections:
- net GND: now also J2.5; no longer J2.4
- net nRF54_RESET: now also J2.3; no longer J2.5
- net nRF54_SWDCLK: now also J2.4; no longer J2.3
- net VOUT1 renamed VOUT2
Changed lines of the file:
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@@
 	(wire
 		(pts
-			(xy 138.43 90.17) (xy 139.7 90.17)
-		)
-		(stroke
-			(width 0)
-			(type default)
-		)
-	)
-	(wire
-		(pts
-			(xy 111.76 85.09) (xy 123.19 85.09)
-		)
-		(stroke
-			(width 0)
-			(type default)
-		)
-	)
-	(wire
-		(pts
-			(xy 118.11 95.25) (xy 125.73 95.25)
-		)
-		(stroke
-			(width 0)
-			(type default)
-		)
-	)
-	(wire
-		(pts
-			(xy 118.11 99.06) (xy 118.11 95.25)
+			(xy 138.43 88.9) (xy 138.43 90.17)
+		)
+		(stroke
+			(width 0)
+			(type default)
+		)
+	)
+	(wire
+		(pts
+			(xy 142.24 92.71) (xy 138.43 92.71)
+		)
+		(stroke
+			(width 0)
+			(type default)
+		)
+	)
+	(wire
+		(pts
+			(xy 123.19 95.25) (xy 125.73 95.25)
+		)
+		(stroke
+			(width 0)
+			(type default)
+		)
+	)
+	(wire
+		(pts
+			(xy 142.24 93.98) (xy 142.24 92.71)
+		)
+		(stroke
+			(width 0)
+			(type default)
+		)
+	)
+	(wire
+		(pts
+			(xy 121.92 92.71) (xy 125.73 92.71)
 		)
 		(stroke
@@
 	(wire
 		(pts
-			(xy 139.7 90.17) (xy 139.7 87.63)
+			(xy 106.68 85.09) (xy 123.19 85.09)
 		)
 		(stroke
@@
 	(wire
 		(pts
-			(xy 118.11 92.71) (xy 125.73 92.71)
-		)
-		(stroke
-			(width 0)
-			(type default)
-		)
-	)
-	(wire
-		(pts
-			(xy 139.7 87.63) (xy 144.78 87.63)
+			(xy 146.05 88.9) (xy 138.43 88.9)
+		)
+		(stroke
+			(width 0)
+			(type default)
+		)
+	)
+	(wire
+		(pts
+			(xy 146.05 93.98) (xy 142.24 93.98)
 		)
 		(stroke
@@
 	(global_label "nRF54_SWDCLK"
 		(shape input)
-		(at 118.11 92.71 180)
+		(at 146.05 93.98 0)
 		(fields_autoplaced yes)
 		(effects
@@
 				(size 1.27 1.27)
 			)
-			(justify right)
+			(justify left)
 		)
 		(property "Intersheetrefs" "${INTERSHEET_REFS}"
-			(at 100.7316 92.71 0)
-			(hide yes)
-			(show_name no)
-			(do_not_autoplace no)
-			(effects
-				(font
-					(size 1.27 1.27)
-				)
-				(justify right)
+			(at 163.4284 93.98 0)
+			(hide yes)
+			(show_name no)
+			(do_not_autoplace no)
+			(effects
+				(font
+					(size 1.27 1.27)
+				)
+				(justify left)
 			)
 		)
@@
 	(global_label "nRF54_SWDIO"
 		(shape input)
-		(at 144.78 87.63 0)
+		(at 146.05 88.9 0)
 		(fields_autoplaced yes)
 		(effects
@@
 		)
 		(property "Intersheetrefs" "${INTERSHEET_REFS}"
-			(at 160.5256 87.63 0)
+			(at 161.7956 88.9 0)
 			(hide yes)
 			(show_name no)
@@
 	(global_label "nRF54_RESET"
 		(shape input)
-		(at 118.11 99.06 180)
+		(at 121.92 92.71 180)
 		(fields_autoplaced yes)
 		(effects
@@
 		)
 		(property "Intersheetrefs" "${INTERSHEET_REFS}"
-			(at 102.4855 99.06 0)
+			(at 106.2955 92.71 0)
 			(hide yes)
 			(show_name no)
@@
 		)
 	)
-	(global_label "VOUT1"
+	(global_label "VOUT2"
 		(shape input)
-		(at 111.76 85.09 180)
+		(at 106.68 85.09 180)
 		(fields_autoplaced yes)
 		(effects
@@
 		)
 		(property "Intersheetrefs" "${INTERSHEET_REFS}"
-			(at 102.8481 85.09 0)
+			(at 97.7681 85.09 0)
 			(hide yes)
 			(show_name no)
@@
 	(symbol
 		(lib_id "power:GND")
-		(at 138.43 92.71 90)
+		(at 123.19 95.25 270)
 		(unit 1)
 		(body_style 1)
@@
 		(in_pos_files yes)
 		(dnp no)
-		(fields_autoplaced yes)
 		(property "Reference" "#PWR031"
-			(at 144.78 92.71 0)
+			(at 116.84 95.25 0)
 			(hide yes)
 			(show_name no)
@@
 		)
 		(property "Value" "GND"
-			(at 142.24 92.7099 90)
-			(show_name no)
-			(do_not_autoplace no)
-			(effects
-				(font
-					(size 1.27 1.27)
-				)
-				(justify right)
+			(at 123.698 97.282 90)
+			(show_name no)
+			(do_not_autoplace no)
+			(effects
+				(font
+					(size 1.27 1.27)
+				)
 			)
 		)
 		(property "Footprint" ""
-			(at 138.43 92.71 0)
+			(at 123.19 95.25 0)
 			(hide yes)
 			(show_name no)
@@
 		)
 		(property "Datasheet" ""
-			(at 138.43 92.71 0)
+			(at 123.19 95.25 0)
 			(hide yes)
 			(show_name no)
@@
 		)
 		(property "Description" "Power symbol creates a global label with name \"GND\" , ground"
-			(at 138.43 92.71 0)
-			(hide yes)
-			(show_name no)
+			(at 123.19 95.25 0)
+			(hide yes)
+			(show_name no)
