File: npm1300.kicad_sch (KiCad schematic)
At the start: 19 parts, among them U2 nPM1300-QEXX

Commit message: Push current KiCad workspace changes
Connections:
- net VOUT2 is gone; now on net VDDIO: C17.2, L10.2, U2.32 (VOUT2)
- net VBAT: no longer U2.15 (SHPHLD)
- net PMIC_INT: now reaches U2.8 (GPIO1)
- no-connect marks 11 -> 10
Changed lines of the file:
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@@
 	)
 	(junction
-		(at 204.47 138.43)
+		(at 111.76 36.83)
 		(diameter 0)
 		(color 0 0 0 0)
@@
 	)
 	(junction
+		(at 200.66 125.73)
+		(diameter 0)
+		(color 0 0 0 0)
+	)
+	(junction
 		(at 196.85 102.87)
 		(diameter 0)
@@
 	)
 	(junction
-		(at 204.47 125.73)
-		(diameter 0)
-		(color 0 0 0 0)
-	)
-	(junction
 		(at 80.01 62.23)
 		(diameter 0)
@@
 	)
 	(no_connect
-		(at 102.87 95.25)
-	)
-	(no_connect
 		(at 102.87 102.87)
 	)
@@
 	(wire
 		(pts
-			(xy 101.6 123.19) (xy 102.87 123.19)
+			(xy 158.75 39.37) (xy 158.75 36.83)
 		)
 		(stroke
@@
 	(wire
 		(pts
-			(xy 158.75 39.37) (xy 158.75 36.83)
+			(xy 93.98 82.55) (xy 102.87 82.55)
 		)
 		(stroke
@@
 	(wire
 		(pts
-			(xy 93.98 82.55) (xy 102.87 82.55)
+			(xy 96.52 100.33) (xy 96.52 95.25)
 		)
 		(stroke
@@
 	(wire
 		(pts
+			(xy 111.76 26.67) (xy 111.76 36.83)
+		)
+		(stroke
+			(width 0)
+			(type default)
+		)
+	)
+	(wire
+		(pts
 			(xy 127 33.02) (xy 128.27 33.02)
 		)
@@
 	(wire
 		(pts
-			(xy 204.47 125.73) (xy 205.74 125.73)
+			(xy 118.11 36.83) (xy 118.11 48.26)
 		)
 		(stroke
@@
 	(wire
 		(pts
-			(xy 118.11 36.83) (xy 118.11 48.26)
+			(xy 214.63 85.09) (xy 214.63 82.55)
 		)
 		(stroke
@@
 	(wire
 		(pts
-			(xy 214.63 85.09) (xy 214.63 82.55)
+			(xy 231.14 64.77) (xy 214.63 64.77)
 		)
 		(stroke
@@
 	(wire
 		(pts
-			(xy 231.14 64.77) (xy 214.63 64.77)
+			(xy 200.66 125.73) (xy 200.66 130.81)
 		)
 		(stroke
@@
 	(wire
 		(pts
-			(xy 194.31 83.82) (xy 200.66 83.82)
+			(xy 77.47 100.33) (xy 96.52 100.33)
 		)
 		(stroke
@@
 	(wire
 		(pts
-			(xy 90.17 123.19) (xy 96.52 123.19)
+			(xy 194.31 83.82) (xy 200.66 83.82)
 		)
 		(stroke
@@
 	(wire
 		(pts
-			(xy 87.63 87.63) (xy 93.98 87.63)
+			(xy 90.17 123.19) (xy 96.52 123.19)
 		)
 		(stroke
@@
 	(wire
 		(pts
-			(xy 173.99 128.27) (xy 173.99 130.81)
+			(xy 87.63 87.63) (xy 93.98 87.63)
 		)
 		(stroke
@@
 	(wire
 		(pts
-			(xy 147.32 22.86) (xy 156.21 22.86)
+			(xy 173.99 128.27) (xy 173.99 130.81)
 		)
 		(stroke
@@
 	(wire
 		(pts
-			(xy 180.34 43.18) (xy 180.34 29.21)
+			(xy 147.32 22.86) (xy 156.21 22.86)
 		)
 		(stroke
@@
 	(wire
 		(pts
-			(xy 158.75 36.83) (xy 156.21 36.83)
+			(xy 180.34 43.18) (xy 180.34 29.21)
 		)
 		(stroke
@@
 	(wire
 		(pts
-			(xy 101.6 148.59) (xy 204.47 148.59)
+			(xy 158.75 36.83) (xy 156.21 36.83)
 		)
 		(stroke
@@
 	(wire
 		(pts
-			(xy 204.47 138.43) (xy 204.47 125.73)
-		)
-		(stroke
-			(width 0)
-			(type default)
-		)
-	)
-	(wire
-		(pts
 			(xy 179.07 52.07) (xy 193.04 52.07)
 		)
@@
 	(wire
 		(pts
-			(xy 101.6 123.19) (xy 101.6 148.59)
-		)
-		(stroke
-			(width 0)
-			(type default)
-		)
-	)
-	(wire
-		(pts
 			(xy 173.99 95.25) (xy 179.07 95.25)
 		)
@@
 	(wire
 		(pts
-			(xy 186.69 125.73) (xy 204.47 125.73)
+			(xy 186.69 125.73) (xy 200.66 125.73)
 		)
 		(stroke
@@
 	(wire
 		(pts
+			(xy 111.76 36.83) (xy 118.11 36.83)
+		)
+		(stroke
+			(width 0)
+			(type default)
+		)
+	)
+	(wire
+		(pts
 			(xy 67.31 59.69) (xy 74.93 59.69)
 		)
@@
 	(wire
 		(pts
-			(xy 106.68 36.83) (xy 118.11 36.83)
+			(xy 106.68 36.83) (xy 111.76 36.83)
 		)
 		(stroke
@@
 	(wire
 		(pts
-			(xy 204.47 148.59) (xy 204.47 138.43)
+			(xy 102.87 107.95) (xy 92.71 107.95)
 		)
 		(stroke
@@
 	(wire
 		(pts
-			(xy 102.87 107.95) (xy 92.71 107.95)
+			(xy 96.52 95.25) (xy 102.87 95.25)
 		)
 		(stroke
@@
 	(wire
 		(pts
+			(xy 200.66 125.73) (xy 205.74 125.73)
+		)
+		(stroke
+			(width 0)
+			(type default)
+		)
+	)
+	(wire
+		(pts
 			(xy 74.93 59.69) (xy 80.01 59.69)
 		)
@@
 		)
 	)
+	(global_label "VOUT2"
+		(shape input)
+		(at 111.76 26.67 0)
+		(fields_autoplaced yes)
+		(effects
+			(font
+				(size 1.27 1.27)
+			)
+			(justify left)
+		)
+		(property "Intersheetrefs" "${INTERSHEET_REFS}"
+			(at 120.6719 26.67 0)
+			(hide yes)
+			(show_name no)
+			(do_not_autoplace no)
+			(effects
+				(font
+					(size 1.27 1.27)
+				)
+				(justify left)
+			)
+		)
+	)
 	(global_label "VDDIO"
 		(shape input)
@@
 		)
 	)
+	(global_label "PMIC_INT"
+		(shape output)
+		(at 77.47 100.33 180)
+		(fields_autoplaced yes)
+		(effects
+			(font
+				(size 1.27 1.27)
+			)
+			(justify right)
+		)
+		(property "Intersheetrefs" "${INTERSHEET_REFS}"
+			(at 66.0181 100.33 0)
+			(hide yes)
+			(show_name no)
+			(do_not_autoplace no)
+			(effects
+				(font
+					(size 1.27 1.27)
+				)
+				(justify right)
+			)
+		)
+	)
 	(global_label "CC2"
 		(shape input)
@@
 	(symbol
 		(lib_id "power:PWR_FLAG")
-		(at 204.47 138.43 270)
+		(at 200.66 130.81 180)
 		(unit 1)
 		(body_style 1)
@@
 		(fields_autoplaced yes)
 		(property "Reference" "#FLG03"
-			(at 206.375 138.43 0)
+			(at 200.66 132.715 0)
 			(hide yes)
 			(show_name no)
@@
 		)
 		(property "Value" "PWR_FLAG"
-			(at 208.28 138.4299 90)
+			(at 203.2 132.0799 0)
 			(show_name no)
 			(do_not_autoplace no)
@@
 					(size 1.27 1.27)
 				)
-				(justify left)
+				(justify right)
 			)
 		)
 		(property "Footprint" ""
-			(at 204.47 138.43 0)
+			(at 200.66 130.81 0)
 			(hide yes)
 			(show_name no)
@@
 		)
 		(property "Datasheet" ""
-			(at 204.47 138.43 0)
+			(at 200.66 130.81 0)
 			(hide yes)
 			(show_name no)
@@
 		)
 		(property "Description" "Special symbol for telling ERC where power comes from"
-			(at 204.47 138.43 0)
+			(at 200.66 130.81 0)
 			(hide yes)
 			(show_name no)
