File: npm1300.kicad_sch (KiCad schematic)
At the start: 19 parts, among them U2 nPM1300-QEXX

Commit message: Update schematic and PCB files
Parts:
- removed R13, R14: 4.7k, Resistor_SMD:R_0402_1005Metric, symbol Device:R
- removed R15: 560, Resistor_SMD:R_0402_1005Metric, symbol Device:R
- removed R8: 10k, Resistor_SMD:R_0402_1005Metric, symbol Device:R
- added R12, R13: 4.7k, easyeda2kicad:R0402, symbol EasyEDA2Kicad:RC0402FR-074K7L
- added R14: 560, easyeda2kicad:R0402, symbol EasyEDA2Kicad:FRC0402F5600TS
- added R8: 10k, easyeda2kicad:R0402, symbol EasyEDA2Kicad:RT0402BRD0710KL
Connections:
- net GND: now also R8.1
- net I2C_SCL: now also R12.1
- net I2C_SDA: now also R13.1
- net VDDIO: now also R12.2, R13.2
- net VSYS: now also R14.2
- net at U2.18 (NTC): now also R8.2
- net at LED1.2 (A): now also R14.1

Commit message: Update KiCad schematic and PCB files
Connections:
- net VBUS renamed CHG_IN
Other:
- note added: "CHG_IN connects to the solar charger and USB"
- note removed: "VBUS connects to the solar charger and USB"
Changed lines of the file:
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@@
 		)
 	)
-	(text "VBUS connects to the solar charger and USB"
+	(text "CHG_IN connects to the solar charger and USB"
 		(exclude_from_sim no)
 		(at 107.442 57.912 0)
@@
 		)
 	)
-	(global_label "VBUS"
+	(global_label "CHG_IN"
 		(shape input)
 		(at 67.31 59.69 180)
@@
 		)
 		(property "Intersheetrefs" "${INTERSHEET_REFS}"
-			(at 59.4262 59.69 0)
+			(at 57.5514 59.69 0)
 			(hide yes)
 			(show_name no)
