File: power_supply.kicad_sch (KiCad schematic)
At the start: 11 parts, among them U3 SPV1040T

Commit message: Save workspace changes
Parts:
- added D2: SS14_C83852, easyeda2kicad:SMA_L4.3-W2.6-LS5.2-RD, symbol EasyEDA2Kicad:SS14_C83852
- added U5: S2B-PH-K-S-GW, easyeda2kicad:CONN-TH_S2B-PH-K-S-GW, symbol EasyEDA2Kicad:S2B-PH-K-S-GW
- L1: value SDFL2012S100KTF -> 10uh
- R6: value 3.9M -> 3.01M
Connections:
- net GND: now also C27.1, U5.2; no longer C27.2
- net SOLAR_5p5V: now also C27.2, R4.1, D2.2 (A), U5.1; no longer C27.1
- net SPV1040T_VOUT: now also D2.1 (K); no longer L1.2, R4.1, U3.3 (LX)
- new net: L1.2, U3.3 (LX)
Other:
- moved on the sheet: C2, C27, D1

Commit message: Update schematic and PCB files
Parts:
- removed R4: 3.3M, Resistor_SMD:R_0402_1005Metric, symbol Device:R
- removed R5, R7: 1M, Resistor_SMD:R_0402_1005Metric, symbol Device:R
- removed R6: 3.01M, Resistor_SMD:R_0402_1005Metric, symbol Device:R
- added R4: 3.3M, easyeda2kicad:R0402, symbol EasyEDA2Kicad:1RC0402J0335
- added R5, R7: 1M, easyeda2kicad:R0402, symbol EasyEDA2Kicad:RC0402JR-071ML
- added R6: 3.01M, easyeda2kicad:R0402, symbol EasyEDA2Kicad:FRC0402F3904TS
Connections:
- net GND: now also R5.1, R7.1
- net SOLAR_5p5V: now also R4.2
- net SPV1040T_VOUT: now also R6.2
- net at C28.2, U3.1 (MPP-SET): now also R4.1, R5.2
- net at U3.5 (VCTRL): now also R6.1, R7.2

Commit message: Update KiCad schematic and PCB files
Connections:
- net VBUS: now also D1.2 (A); no longer D1.1 (K)
- net SPV1040T_VOUT renamed CHG_IN
- net CHG_IN: now also D1.1 (K); no longer D1.2 (A)
Other:
- moved on the sheet: D1
Changed lines of the file:
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@@
-	)
-	(junction
-		(at 168.91 82.55)
-		(diameter 0)
-		(color 0 0 0 0)
 	)
 	(junction
@@
 		(color 0 0 0 0)
 	)
+	(junction
+		(at 88.9 144.78)
+		(diameter 0)
+		(color 0 0 0 0)
+	)
 	(wire
 		(pts
@@
 	(wire
 		(pts
+			(xy 88.9 97.79) (xy 78.74 97.79)
+		)
+		(stroke
+			(width 0)
+			(type default)
+		)
+	)
+	(wire
+		(pts
 			(xy 107.95 144.78) (xy 127 144.78)
 		)
@@
 	(wire
 		(pts
-			(xy 88.9 97.79) (xy 78.74 97.79)
-		)
-		(stroke
-			(width 0)
-			(type default)
-		)
-	)
-	(wire
-		(pts
 			(xy 119.38 92.71) (xy 119.38 90.17)
 		)
@@
 	(wire
 		(pts
-			(xy 168.91 90.17) (xy 168.91 82.55)
+			(xy 168.91 78.74) (xy 168.91 90.17)
 		)
 		(stroke
@@
 	(wire
 		(pts
-			(xy 168.91 82.55) (xy 168.91 78.74)
-		)
-		(stroke
-			(width 0)
-			(type default)
-		)
-	)
-	(wire
-		(pts
 			(xy 162.56 67.31) (xy 162.56 59.69)
 		)
@@
 	(wire
 		(pts
+			(xy 88.9 144.78) (xy 97.79 144.78)
+		)
+		(stroke
+			(width 0)
+			(type default)
+		)
+	)
+	(wire
+		(pts
 			(xy 184.15 93.98) (xy 184.15 96.52)
 		)
@@
 	(wire
 		(pts
-			(xy 86.36 144.78) (xy 97.79 144.78)
+			(xy 86.36 144.78) (xy 88.9 144.78)
 		)
 		(stroke
@@
 		)
 	)
-	(global_label "SPV1040T_VOUT"
+	(global_label "CHG_IN"
 		(shape input)
 		(at 76.2 119.38 180)
@@
 		)
 		(property "Intersheetrefs" "${INTERSHEET_REFS}"
-			(at 58.1563 119.38 0)
+			(at 66.4414 119.38 0)
 			(hide yes)
 			(show_name no)
@@
 		)
 	)
-	(global_label "SPV1040T_VOUT"
+	(global_label "CHG_IN"
 		(shape input)
 		(at 190.5 76.2 0)
@@
 		)
 		(property "Intersheetrefs" "${INTERSHEET_REFS}"
-			(at 208.5437 76.2 0)
+			(at 200.2586 76.2 0)
 			(hide yes)
 			(show_name no)
@@
 		)
 	)
-	(global_label "SPV1040T_VOUT"
+	(global_label "CHG_IN"
 		(shape input)
 		(at 166.37 59.69 0)
@@
 		)
 		(property "Intersheetrefs" "${INTERSHEET_REFS}"
-			(at 184.4137 59.69 0)
+			(at 176.1286 59.69 0)
 			(hide yes)
 			(show_name no)
@@
 	(symbol
 		(lib_id "power:PWR_FLAG")
-		(at 168.91 82.55 270)
+		(at 88.9 144.78 180)
 		(unit 1)
 		(body_style 1)
@@
 		(fields_autoplaced yes)
 		(property "Reference" "#FLG01"
-			(at 170.815 82.55 0)
+			(at 88.9 146.685 0)
 			(hide yes)
 			(show_name no)
@@
 		)
 		(property "Value" "PWR_FLAG"
-			(at 172.72 82.5499 90)
-			(show_name no)
-			(do_not_autoplace no)
-			(effects
-				(font
-					(size 1.27 1.27)
-				)
-				(justify left)
+			(at 91.44 146.0499 0)
+			(show_name no)
+			(do_not_autoplace no)
+			(effects
+				(font
+					(size 1.27 1.27)
+				)
+				(justify right)
 			)
 		)
 		(property "Footprint" ""
-			(at 168.91 82.55 0)
+			(at 88.9 144.78 0)
 			(hide yes)
 			(show_name no)
@@
 		)
 		(property "Datasheet" ""
-			(at 168.91 82.55 0)
+			(at 88.9 144.78 0)
 			(hide yes)
 			(show_name no)
@@
 		)
 		(property "Description" "Special symbol for telling ERC where power comes from"
-			(at 168.91 82.55 0)
+			(at 88.9 144.78 0)
 			(hide yes)
 			(show_name no)
@@
 	(symbol
 		(lib_id "EasyEDA2Kicad:SS14_C83852")
-		(at 102.87 144.78 0)
+		(at 102.87 144.78 180)
 		(unit 1)
 		(body_style 1)
@@
 		(fields_autoplaced yes)
 		(property "Reference" "D1"
-			(at 102.49 138.43 0)
+			(at 103.25 138.43 0)
 			(show_name no)
 			(do_not_autoplace no)
@@
 		)
 		(property "Value" "SS14_C83852"
-			(at 102.49 140.97 0)
+			(at 103.25 140.97 0)
 			(show_name no)
 			(do_not_autoplace no)
@@
 		)
 		(property "Footprint" "easyeda2kicad:SMA_L4.3-W2.6-LS5.2-RD"
-			(at 102.87 152.4 0)
+			(at 102.87 137.16 0)
 			(hide yes)
 			(show_name no)
@@
 		)
 		(property "Datasheet" "https://lcsc.com/product-detail/Schottky-Barrier-Diodes-SBD_ON-Semicon_SS14_ON-Semicon-ON-SS14_C83852.html"
-			(at 102.87 154.94 0)
+			(at 102.87 134.62 0)
 			(hide yes)
 			(show_name no)
@@
 		)
 		(property "Manufacturer" "onsemi(安森美)"
-			(at 102.87 157.48 0)
+			(at 102.87 132.08 0)
 			(hide yes)
 			(show_name no)
@@
 		)
 		(property "MPN" "SS14"
-			(at 102.87 160.02 0)
+			(at 102.87 129.54 0)
 			(hide yes)
 			(show_name no)
@@
 		)
 		(property "LCSC Part" "C83852"
-			(at 102.87 162.56 0)
-			(hide yes)
-			(show_name no)
+			(at 102.87 127 0)
+			(hide yes)
+			(show_name no)
