File: usb.kicad_sch (KiCad schematic)
At the start: 4 parts, among them J3 USB_C_Receptacle_PowerOnly_6P

Commit message: Update schematic and PCB files
Parts:
- removed R1, R2: 5.1k, EasyEDA2Kicad:R0402, symbol PCM_Resistor_US_AKL:R_Generic
- added J1: TYPE-C-31-M-12, TYPE-C-31-M-12:HRO_TYPE-C-31-M-12, symbol TYPE-C-31-M-12:TYPE-C-31-M-12
- added R1, R2: 5.1k, easyeda2kicad:R0402, symbol EasyEDA2Kicad:RCA025K1FLF
Connections:
- net CC1: now also R2.2
- net CC2: now also R1.2
- net GND: now also J1.A1_B12 (GND), J1.B1_A12 (GND), R1.1, R2.1
- net VBUS: now also J1.A4_B9 (VBUS), J1.B4_A9 (VBUS)
- new net: J1.S1 (SHIELD), J1.S2 (SHIELD), J1.S3 (SHIELD), J1.S4 (SHIELD)

Commit message: Update KiCad schematic and PCB files
Parts:
- removed J3: USB_C_Receptacle_PowerOnly_6P, Connector_USB:USB_C_Receptacle_HRO_TYPE-C-31-M-12, symbol Connector:USB_C_Receptacle_PowerOnly_6P
- J1: footprint TYPE-C-31-M-12:HRO_TYPE-C-31-M-12 -> easyeda2kicad:USB-C_SMD-TYPE-C-31-M-12_1
Connections:
- net CC1: now also J1.A5 (CC1)
- net CC2: now also J1.B5 (CC2)
- net GND: now also J1.S1 (SHIELD), J1.S2 (SHIELD), J1.S3 (SHIELD), J1.S4 (SHIELD)
Other:
- moved on the sheet: J1
