File: nrf54l15_v4/nrf54l15_v4/antenna.kicad_sch (KiCad schematic)
At the start: 7 parts

Commit message: Update nrf54l15_v4 design; add feather board, enclosure, and docs
nrf54l15_v4:
- Sensor connector (CN1) reworked to a 14-pin Molex 503480-1400 FFC
  connector with a project footprint library (nrf54l15_v4.pretty) and
  vendor drawing/3D model.
- nRF54L15 pin assignment fixes for the sensor bus (I2C, SPI/UART, INT,
  AIN, board-ID).
- AEM10330 solar block: EN_SLEEP tied to GND, MPPT ratio set to 70%,
  MPNs added to C40-C43.
- Annotation cleanup across antenna, npm1300 and power_supply sheets;
  PCB updated from schematic; zone min clearance set to 0.5 mm.
- Add 3D-printable enclosure generator and STL outputs.

New:
- nrf54l15_feather KiCad project.
- Sensor_Boards/Conductivity_Salinity design notes.
- solar-analysis-v4.md and v4-sensor-connector.md design docs.
- AEM10330 and PowerFilm LL200-2.4-75 datasheets.

Other:
- nrf54l15_v2 BOM: fix misplaced capacitance value columns (C9/C11);
  add .xlsx BOM.
- .gitignore: ignore dated schematic backups, extra claude_bak copies,
  vendor zip downloads and DRC report exports.

Co-Authored-By: Claude Opus 5.5 <noreply@anthropic.com>
Connections:
- net GND: no longer AE1.2
- no-connect marks 0 -> 1
Changed lines of the file:
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@@
 		(color 0 0 0 0)
+	)
+	(no_connect
+		(at 55.88 123.19)
 	)
 	(wire
@@
 			)
 		)
-	)
-	(symbol
-		(lib_id "power:GND")
-		(at 55.88 123.19 0)
-		(unit 1)
-		(body_style 1)
-		(exclude_from_sim no)
-		(in_bom yes)
-		(on_board yes)
-		(in_pos_files yes)
-		(dnp no)
-		(fields_autoplaced yes)
-		(property "Reference" "#PWR042"
-			(at 55.88 129.54 0)
-			(hide yes)
-			(show_name no)
-			(do_not_autoplace no)
-			(effects
-				(font
-					(size 1.27 1.27)
-				)
-			)
-		)
-		(property "Value" "GND"
-			(at 55.88 128.27 0)
-			(show_name no)
-			(do_not_autoplace no)
-			(effects
-				(font
-					(size 1.27 1.27)
-				)
-			)
-		)
-		(property "Footprint" ""
-			(at 55.88 123.19 0)
-			(hide yes)
-			(show_name no)
-			(do_not_autoplace no)
-			(effects
-				(font
-					(size 1.27 1.27)
-				)
-			)
-		)
-		(property "Datasheet" ""
-			(at 55.88 123.19 0)
-			(hide yes)
-			(show_name no)
-			(do_not_autoplace no)
-			(effects
-				(font
-					(size 1.27 1.27)
-				)
-			)
-		)
-		(property "Description" "Power symbol creates a global label with name \"GND\" , ground"
-			(at 55.88 123.19 0)
-			(hide yes)
-			(show_name no)
-			(do_not_autoplace no)
-			(effects
-				(font
-					(size 1.27 1.27)
-				)
-			)
-		)
-		(pin "1"
-		)
-		(instances
-			(project "nrf54l15_v4"
-				(path "/55da176d-6431-4d58-ada7-b89d931b1434/1978a031-5300-455a-be04-a92eb95c93f3"
-					(reference "#PWR042")
-					(unit 1)
-				)
-			)
-		)
