File: nrf54l15_v4/nrf54l15_v4/npm1300.kicad_sch (KiCad schematic)
At the start: 20 parts, among them U2 nPM1300-QEXX

Commit message: Update nrf54l15_v4 design; add feather board, enclosure, and docs
nrf54l15_v4:
- Sensor connector (CN1) reworked to a 14-pin Molex 503480-1400 FFC
  connector with a project footprint library (nrf54l15_v4.pretty) and
  vendor drawing/3D model.
- nRF54L15 pin assignment fixes for the sensor bus (I2C, SPI/UART, INT,
  AIN, board-ID).
- AEM10330 solar block: EN_SLEEP tied to GND, MPPT ratio set to 70%,
  MPNs added to C40-C43.
- Annotation cleanup across antenna, npm1300 and power_supply sheets;
  PCB updated from schematic; zone min clearance set to 0.5 mm.
- Add 3D-printable enclosure generator and STL outputs.

New:
- nrf54l15_feather KiCad project.
- Sensor_Boards/Conductivity_Salinity design notes.
- solar-analysis-v4.md and v4-sensor-connector.md design docs.
- AEM10330 and PowerFilm LL200-2.4-75 datasheets.

Other:
- nrf54l15_v2 BOM: fix misplaced capacitance value columns (C9/C11);
  add .xlsx BOM.
- .gitignore: ignore dated schematic backups, extra claude_bak copies,
  vendor zip downloads and DRC report exports.

Co-Authored-By: Claude Opus 5.5 <noreply@anthropic.com>
Connections:
- net VDDIO: now also U2.28 (LSIN1/VINLDO1)
- net VSENS: now reaches U2.29 (LSOUT1/VOUTLDO1)
- no-connect marks 10 -> 8
Other:
- note added: "LDSW1 is the sensor load switch. LSIN1 = VOUT2, LSOUT1 = VSENS. Configure as a load switch, not an LDO."
Changed lines of the file:
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@@
+		)
+	)
+	(text "LDSW1 is the sensor load switch. LSIN1 = VOUT2, LSOUT1 = VSENS. Configure as a load switch, not an LDO."
+		(exclude_from_sim no)
+		(at 170.434 155.448 0)
+		(effects
+			(font
+				(size 1.27 1.27)
+			)
 		)
 	)
 	(text "VBUS: USB-C input only (solar charges VBAT directly via AEM10330 on power_supply sheet)"
 		(exclude_from_sim no)
-		(at 107.442 57.912 0)
+		(at 71.628 20.574 0)
 		(effects
 			(font
@@
 	)
 	(junction
+		(at 181.61 90.17)
+		(diameter 0)
+		(color 0 0 0 0)
+	)
+	(junction
 		(at 196.85 102.87)
 		(diameter 0)
@@
 	)
 	(no_connect
-		(at 173.99 102.87)
-	)
-	(no_connect
 		(at 173.99 110.49)
-	)
-	(no_connect
-		(at 173.99 105.41)
 	)
 	(no_connect
@@
 	(wire
 		(pts
+			(xy 173.99 105.41) (xy 203.2 105.41)
+		)
+		(stroke
+			(width 0)
+			(type default)
+		)
+	)
+	(wire
+		(pts
 			(xy 118.11 36.83) (xy 118.11 48.26)
 		)
@@
 	(wire
 		(pts
+			(xy 181.61 90.17) (xy 181.61 102.87)
+		)
+		(stroke
+			(width 0)
+			(type default)
+		)
+	)
+	(wire
+		(pts
 			(xy 96.52 95.25) (xy 102.87 95.25)
 		)
@@
 		(pts
 			(xy 140.97 43.18) (xy 180.34 43.18)
+		)
+		(stroke
+			(width 0)
+			(type default)
+		)
+	)
+	(wire
+		(pts
+			(xy 181.61 102.87) (xy 173.99 102.87)
 		)
 		(stroke
@@
 			)
 		)
+	)
+	(global_label "VSENS"
+		(shape input)
+		(at 203.2 105.41 0)
+		(fields_autoplaced yes)
+		(effects
+			(font
+				(size 1.27 1.27)
+			)
+			(justify left)
+		)
+		(property "Intersheetrefs" "${INTERSHEET_REFS}"
+			(at 203.2 105.41 0)
+			(hide yes)
+			(show_name no)
+			(do_not_autoplace no)
+			(effects
+				(font
+					(size 1.27 1.27)
+				)
+				(justify left)
+			)
+		)
