File: nrf54l15_v4/nrf54l15_v4/power_supply.kicad_sch (KiCad schematic)
At the start: 7 parts, among them IC1 AEM10330-QFN, U5 S2B-PH-K-S-GW

Commit message: Update nrf54l15_v4 design; add feather board, enclosure, and docs
nrf54l15_v4:
- Sensor connector (CN1) reworked to a 14-pin Molex 503480-1400 FFC
  connector with a project footprint library (nrf54l15_v4.pretty) and
  vendor drawing/3D model.
- nRF54L15 pin assignment fixes for the sensor bus (I2C, SPI/UART, INT,
  AIN, board-ID).
- AEM10330 solar block: EN_SLEEP tied to GND, MPPT ratio set to 70%,
  MPNs added to C40-C43.
- Annotation cleanup across antenna, npm1300 and power_supply sheets;
  PCB updated from schematic; zone min clearance set to 0.5 mm.
- Add 3D-printable enclosure generator and STL outputs.

New:
- nrf54l15_feather KiCad project.
- Sensor_Boards/Conductivity_Salinity design notes.
- solar-analysis-v4.md and v4-sensor-connector.md design docs.
- AEM10330 and PowerFilm LL200-2.4-75 datasheets.

Other:
- nrf54l15_v2 BOM: fix misplaced capacitance value columns (C9/C11);
  add .xlsx BOM.
- .gitignore: ignore dated schematic backups, extra claude_bak copies,
  vendor zip downloads and DRC report exports.

Co-Authored-By: Claude Opus 5.5 <noreply@anthropic.com>
Parts:
- C40: MPN (none) -> GRM188R61A226ME15; Manufacturer (none) -> Murata
- C41: MPN (none) -> GRM155R60J106ME15; Manufacturer (none) -> Murata
- C42: MPN (none) -> GRM188R60J476ME15; Manufacturer (none) -> Murata
- C43: MPN (none) -> MSASJ31LBB5227MTCA01; Manufacturer (none) -> Taiyo Yuden
Connections:
- net GND: now also IC1.11 (R_MPP[2]), IC1.39 (EN_SLEEP); no longer IC1.12 (R_MPP[1])
- net LOAD: no longer IC1.39 (EN_SLEEP)
- net VINT: now also IC1.12 (R_MPP[1]); no longer IC1.11 (R_MPP[2])
Changed lines of the file:
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@@
 		)
 	)
-	(label "GND"
+	(label "VINT"
 		(at 120.65 127 270)
 		(effects
@@
 		)
 	)
-	(label "LOAD"
-		(at 123.19 55.88 90)
-		(effects
-			(font
-				(size 1.27 1.27)
-			)
-			(justify left bottom)
-		)
-	)
 	(label "GND"
 		(at 138.43 55.88 90)
@@
 		)
 	)
-	(label "VINT"
+	(label "GND"
 		(at 118.11 127 270)
 		(effects
@@
 	)
 	(symbol
+		(lib_id "power:GND")
+		(at 123.19 55.88 180)
+		(unit 1)
+		(body_style 1)
+		(exclude_from_sim no)
+		(in_bom yes)
+		(on_board yes)
+		(in_pos_files yes)
+		(dnp no)
+		(fields_autoplaced yes)
+		(property "Reference" "#PWR04"
+			(at 123.19 49.53 0)
+			(hide yes)
+			(show_name no)
+			(do_not_autoplace no)
+			(effects
+				(font
+					(size 1.27 1.27)
+				)
+			)
+		)
+		(property "Value" "GND"
+			(at 123.19 50.8 0)
+			(show_name no)
+			(do_not_autoplace no)
+			(effects
+				(font
+					(size 1.27 1.27)
+				)
+			)
+		)
+		(property "Footprint" ""
+			(at 123.19 55.88 0)
+			(hide yes)
+			(show_name no)
+			(do_not_autoplace no)
+			(effects
+				(font
+					(size 1.27 1.27)
+				)
+			)
+		)
+		(property "Datasheet" ""
+			(at 123.19 55.88 0)
+			(hide yes)
+			(show_name no)
+			(do_not_autoplace no)
+			(effects
+				(font
+					(size 1.27 1.27)
+				)
+			)
+		)
+		(property "Description" "Power symbol creates a global label with name \"GND\" , ground"
+			(at 123.19 55.88 0)
+			(hide yes)
+			(show_name no)
+			(do_not_autoplace no)
+			(effects
+				(font
+					(size 1.27 1.27)
+				)
+			)
+		)
+		(pin "1"
+		)
+		(instances
+			(project "nrf54l15_v4"
+				(path "/55da176d-6431-4d58-ada7-b89d931b1434/7400a6e7-510a-4e28-84b8-c443b681fae8"
+					(reference "#PWR04")
+					(unit 1)
+				)
+			)
+		)
+	)
+	(symbol
 		(lib_id "Device:L")
 		(at 180.34 130.81 0)
@@
 			)
 		)
+		(property "Manufacturer" "Murata"
+			(at 191.77 107.95 0)
+			(hide yes)
+			(show_name no)
+			(do_not_autoplace no)
+			(effects
+				(font
+					(size 1.27 1.27)
+				)
+			)
+		)
+		(property "MPN" "GRM155R60J106ME15"
+			(at 191.77 107.95 0)
+			(hide yes)
+			(show_name no)
+			(do_not_autoplace no)
+			(effects
+				(font
+					(size 1.27 1.27)
+				)
+			)
+		)
 		(pin "1"
 		)
@@
 			)
 		)
+		(property "Manufacturer" "Murata"
+			(at 180.34 64.77 0)
+			(hide yes)
+			(show_name no)
+			(do_not_autoplace no)
+			(effects
+				(font
+					(size 1.27 1.27)
+				)
+			)
+		)
+		(property "MPN" "GRM188R61A226ME15"
+			(at 180.34 64.77 0)
+			(hide yes)
+			(show_name no)
+			(do_not_autoplace no)
+			(effects
+				(font
+					(size 1.27 1.27)
+				)
+			)
+		)
 		(pin "1"
 		)
@@
 		(property "Description" ""
 			(at 208.28 106.68 0)
+			(show_name no)
+			(do_not_autoplace no)
+			(effects
+				(font
+					(size 1.27 1.27)
+				)
+			)
+		)
+		(property "Manufacturer" "Murata"
+			(at 208.28 106.68 0)
+			(hide yes)
+			(show_name no)
+			(do_not_autoplace no)
+			(effects
+				(font
+					(size 1.27 1.27)
+				)
+			)
+		)
+		(property "MPN" "GRM188R60J476ME15"
+			(at 208.28 106.68 0)
+			(hide yes)
 			(show_name no)
 			(do_not_autoplace no)
@@
 			(show_name no)
 			(do_not_autoplace no)
+			(effects
+				(font
+					(size 1.27 1.27)
+				)
+			)
+		)
+		(property "Manufacturer" "Taiyo Yuden"
+			(at 224.79 106.68 0)
+			(hide yes)
+			(show_name no)
+			(do_not_autoplace no)
+			(effects
+				(font
+					(size 1.27 1.27)
+				)
+			)
+		)
+		(property "MPN" "MSASJ31LBB5227MTCA01"
+			(at 224.79 106.68 0)
+			(hide yes)
+			(show_name no)
+			(do_not_autoplace no)
