File: nrf54l15_feather/nrf54l15_feather/SWD_Debug.kicad_sch (KiCad schematic)
At the start: 1 part, among them J3 FTSH-105-01-L-DV-K

Commit message: Update the nRF54L15 feather and add the feather sens1 and pouch gateway designs.
Co-authored-by: Cursor <cursoragent@cursor.com>
Parts:
- J3: MP FTSH-105-01-L-DV-K -> FTSH-105-01-L-DV-K-TR; MPN (none) -> FTSH-105-01-L-DV-K-TR
