File: nrf54l15_feather/nrf54l15_feather/npm1300.kicad_sch (KiCad schematic)
At the start: 20 parts, among them U2 nPM1300-QEXX

Commit message: Update the nRF54L15 feather and add the feather sens1 and pouch gateway designs.
Co-authored-by: Cursor <cursoragent@cursor.com>
Parts:
- added SW1: SW_Push, Button_Switch_SMD:SW_SPST_B3U-1000P, symbol Switch:SW_Push
- U2: MPN (none) -> nPM1300-QEAA-R7
Connections:
- net GND: now also SW1.1
- net at U2.15 (SHPHLD): now also SW1.2
