File: nrf54l15_feather/nrf54l15_feather/nrf54l15.kicad_sch (KiCad schematic)
At the start: 16 parts, among them U6 nRF54L15-QFXX, X1 XL7EL89CKI-111YLC-32M

Commit message: Update the nRF54L15 feather and add the feather sens1 and pouch gateway designs.
Co-authored-by: Cursor <cursoragent@cursor.com>
Parts:
- U6: MPN (none) -> nRF54L15-QFAA-R
Connections:
- no-connect marks 15 -> 17
