File: nrf54l15_feather/nrf54l15_feather/power_supply.kicad_sch (KiCad schematic)
At the start: 7 parts, among them IC1 AEM10330-QFN, U5 S2B-PH-K-S-GW

Commit message: Update the nRF54L15 feather and add the feather sens1 and pouch gateway designs.
Co-authored-by: Cursor <cursoragent@cursor.com>
Parts:
- C40: MPN GRM188R61A226ME15 -> GRM188R61A226ME15D
- C42: MPN GRM188R60J476ME15 -> GRM188R60J476ME15D
